Commit message: ugv

File: install/my_robot_description/share/my_robot_description/urdf/camera.xacro (robot description, xacro)
@@ -4,5 +4,5 @@
     <xacro:property name="camera_width" value="0.2"/>
     <xacro:property name="camera_height" value="0.12"/>
-    <link name="camera_link">
+    <link name="front_camera_link">
         <visual>
             <geometry>
@@ -21,9 +21,9 @@
      <joint name="base_camera_joint" type="fixed">
         <parent link="base_link"/>
-        <child link="camera_link"/>
+        <child link="front_camera_link"/>
         <!-- <origin xyz="0.6 0 0" rpy="0 0 0"/>   -->
-        <origin xyz="0.8 0 0.3" rpy="0 0 0"/>
+        <origin xyz="0.76 0 0.3" rpy="0 0 0"/>
      </joint>
-     <gazebo reference="camera_link">
+     <gazebo reference="front_camera_link">
         <material>Gazebo/Red</material>
         <sensor name="camera_sensor" type="camera">
@@ -32,5 +32,37 @@
             <update_rate>10.0</update_rate>
             <plugin name="camera_controller" filename="libgazebo_ros_camera.so">
-                <frame_name>camera_link</frame_name>
+                <frame_name>front_camera_link</frame_name>
+            </plugin>
+        </sensor>
+     </gazebo>
+     <link name="back_camera_link">
+        <visual>
+            <geometry>
+                <box size="${camera_length} ${camera_width} ${camera_height}" />
+            </geometry>
+            <material name="black" />
+        </visual>
+        <collision>
+            <geometry>
+                <box size="${camera_length} ${camera_width} ${camera_height}" />
+            </geometry>
+        </collision>
+        <xacro:body_inertia m="0.1" l="${camera_length}" w="${camera_width}" h="${camera_height}"
+                           xyz="0 0 0" rpy="0 0 0" />
+    </link>
+    <joint name="base_camera1_joint" type="fixed">
+        <parent link="base_link"/>
+        <child link="back_camera_link"/>
+        <!-- <origin xyz="0.6 0 0" rpy="0 0 0"/>   -->
+        <origin xyz="-0.96 0 0.3" rpy="0 3.2 0"/>
+     </joint>
+         <gazebo reference="back_camera_link">
+        <material>Gazebo/Red</material>
+        <sensor name="camera_sensor" type="camera">
+            <pose>0 0 0 0 0 0 </pose>
+            <visualize>false</visualize>
+            <update_rate>10.0</update_rate>
+            <plugin name="camera_controller1" filename="libgazebo_ros_camera.so">
+                <frame_name>back_camera_link</frame_name>
             </plugin>
         </sensor>

File: install/my_robot_description/share/my_robot_description/urdf/mobile_base_gazebo.xacro (robot description, xacro)
@@ -6,13 +6,33 @@
     <gazebo reference="right_wheel_link">
         <material>Gazebo/Black</material>
+        <mu1 value="2.0"/>
+    <mu2 value="2.0"/>
+    <kp  value="10000000.0" />
+    <kd  value="1.0" />
+    <fdir1 value="0 1 0"/>
     </gazebo>
     <gazebo reference="left_wheel_link">
         <material>Gazebo/Black</material>
+        <mu1 value="2.0"/>
+    <mu2 value="2.0"/>
+    <kp  value="10000000.0" />
+    <kd  value="1.0" />
+    <fdir1 value="0 1 0"/>
     </gazebo>
      <gazebo reference="back_right_wheel_link">
         <material>Gazebo/Black</material>
+        <mu1 value="2.0"/>
+        <mu2 value="2.0"/>
+        <kp  value="10000000.0" />
+        <kd  value="1.0" />
+        <fdir1 value="0 1 0"/>
     </gazebo>
      <gazebo reference="back_left_wheel_link">
         <material>Gazebo/Black</material>
+        <mu1 value="2.0"/>
+    <mu2 value="2.0"/>
+    <kp  value="10000000.0" />
+    <kd  value="1.0" />
+    <fdir1 value="0 1 0"/>
     </gazebo>
     <gazebo>
@@ -23,5 +43,5 @@
             <!-- <left_joint>base_back_right_wheel_joint</left_joint>
             <right_joint>base_back_left_wheel_joint</right_joint>
-   -->
+    -->
             <wheel_separation>0.60</wheel_separation>
             <wheel_diameter>0.2</wheel_diameter>

File: install/my_robot_description/share/my_robot_description/urdf/ugv.urdf.xacro (robot description, xacro)
@@ -5,4 +5,5 @@
      <xacro:include filename="camera.xacro" />
      <xacro:include filename="lidar.xacro" />
+     <xacro:include filename="ultrasonic.xacro"/>
      <xacro:property name="base_length" value="0.12" />
      <xacro:property name="base_width" value="0.8" />
@@ -115,15 +116,39 @@
         <axis xyz="0 1 0" />
     </joint>
-      <joint name="base_back_right_wheel_joint" type="continuous">
+      <joint name="base_back_right_wheel_joint" type="revolute">
         <parent link="base_link" />
         <child link="back_right_wheel_link" />
         <origin xyz="0.38 -0.480 0.1" rpy="0 0 0" />
-        <axis xyz="0 1 0" />
+        <!-- <axis xyz="0 1 0" /> -->
+        <axis xyz="0.0 0.0 0.1"/>
+        <limit lower="-0.50" upper="0.50" effort="1000" velocity="3"/>
     </joint>
-        <joint name="base_back_left_wheel_joint" type="continuous">
+        <joint name="base_back_left_wheel_joint" type="revolute">
         <parent link="base_link" />
         <child link="back_left_wheel_link" />
         <origin xyz="0.38 0.480 0.1" rpy="0 0 0" />
-        <axis xyz="0 1 0" />
+        <!-- <axis xyz="0 1 0" /> -->
+        <axis xyz="0.0 0.0 0.1"/>
+        <limit lower="-0.50" upper="0.50" effort="1000" velocity="3"/>
     </joint>
+    <transmission name="trans_right_wheel_hing">
+        <type>transmission_interface/SimpleTransmission</type>
+        <joint name="base_back_right_wheel_joint">
+          <hardwareInterface>EffortJointInterface</hardwareInterface>
+        </joint>
+        <actuator name="motor1">
+          <hardwareInterface>EffortJointInterface</hardwareInterface>
+          <mechanicalReduction>1</mechanicalReduction>
+        </actuator>
+      </transmission>
+      <transmission name="trans_right_wheel_rotate">
+        <type>transmission_interface/SimpleTransmission</type>
+        <joint name="base_back_left_wheel_joint">
+          <hardwareInterface>EffortJointInterface</hardwareInterface>
+        </joint>
+        <actuator name="motor_right_wheel_rotate">
+          <hardwareInterface>EffortJointInterface</hardwareInterface>
+          <mechanicalReduction>1</mechanicalReduction>
+        </actuator>
+      </transmission>
 </robot>

File: src/install/my_robot_description/share/my_robot_description/urdf/common_properties.xacro (robot description, xacro)
@@ -6,4 +6,10 @@
         <material name="black">
         <color rgba="0 0 0 1" />
+    </material>
+     <material name="blue">
+        <color rgba="0 0 0.5 1" />
+    </material>
+    <material name="red">
+        <color rgba="1 0 0 1" />
     </material>
         <xacro:macro name="body_inertia" params="m l w h xyz rpy">

File: src/install/my_robot_description/share/my_robot_description/urdf/ugv.urdf.xacro (robot description, xacro)
@@ -2,27 +2,30 @@
 <robot name="my_robot" xmlns:xacro="http://www.ros.org/wiki/xacro">
      <xacro:include filename="common_properties.xacro" />
-     <xacro:property name="base_length" value="1.77" />
-     <xacro:property name="base_height" value="0.63" />
-     <xacro:property name="base_width" value="0.928" />
+     <xacro:include filename="mobile_base_gazebo.xacro" />
+     <xacro:include filename="camera.xacro" />
+     <xacro:include filename="lidar.xacro" />
+     <xacro:property name="base_length" value="0.12" />
+     <xacro:property name="base_width" value="0.8" />
+    <xacro:property name="base_height" value="0.4" />
      <xacro:property name="wheel_radius" value="0.2" />
      <xacro:property name="wheel_length" value="0.10" />
     <link name="base_footprint" />
     <link name="base_link">
-        <visual>
-            <geometry>
-           <box size="1.0 1.0 1.0"/>
-            </geometry>
+       <visual>
+          <geometry>
+                <mesh filename="$(find my_robot_description)/meshes/body1.dae"/>
+                <!-- <mesh filename="package://my_robot_description/meshes/body1.dae"/> -->
+          </geometry>
+            <origin xyz="0 0 -0.1" rpy="0 0 3.14159" />
         </visual>
            <collision>
             <geometry>
-                 <box size="1.0 1.0 1.0"/>
+                    <mesh filename="package://my_robot_description/meshes/body1.dae"/>
+              <!-- <mesh filename="$(find my_robot_description)/meshes/body1.dae"/> -->
             </geometry>
+                <origin xyz="0 0 -0.1" rpy="0 0 3.14159" />
         </collision>
-         <inertial>
-      <mass value="5.0"/>
-      <inertia  ixx="3" ixy="2"  ixz="2"
-                iyy="0.001"  iyz="0.0"
-                izz="0.001"/>
-    </inertial>
+          <xacro:body_inertia m="5.0"  l="0.9" w="0.5" h="0.8"
+                                   xyz="0 0 0" rpy="0 0 0" />
     </link>
     <link name="right_wheel_link">
@@ -41,5 +44,5 @@
                 <origin xyz="0 0 0" rpy="1.57 0 0" />
             </collision>
-          <xacro:cylinder_inertia m="1.0" r="${2*wheel_radius}" h="${2*wheel_length}"
+          <xacro:cylinder_inertia m="1.0" r="${wheel_radius}" h="${wheel_length}"
                                    xyz="0 0 0" rpy="1.57 0 0" />
     </link>
@@ -58,5 +61,5 @@
                 <origin xyz="0 0 0" rpy="1.57 0 0" />
             </collision>
-        <xacro:cylinder_inertia m="1.0" r="${2*wheel_radius}" h="${2*wheel_length}"
+        <xacro:cylinder_inertia m="1.0" r="${wheel_radius}" h="${wheel_length}"
                                    xyz="0 0 0" rpy="1.57 0 0" />
     </link>
@@ -75,5 +78,5 @@
                 <origin xyz="0 0 0" rpy="1.57 0 0" />
             </collision>
-       <xacro:cylinder_inertia m="1.0" r="${2*wheel_radius}" h="${2*wheel_length}"
+       <xacro:cylinder_inertia m="1.0" r="${wheel_radius}" h="${wheel_length}"
                                    xyz="0 0 0" rpy="1.57 0 0" />
     </link>
@@ -92,5 +95,5 @@
                 <origin xyz="0 0 0" rpy="1.57 0 0" />
             </collision>
-          <xacro:cylinder_inertia m="1.0" r="${2*wheel_radius}" h="${2*wheel_length}"
+          <xacro:cylinder_inertia m="1.0" r="${wheel_radius}" h="${wheel_length}"
                                    xyz="0 0 0" rpy="1.57 0 0" />
     </link>
@@ -103,5 +106,5 @@
         <parent link="base_link" />
         <child link="right_wheel_link" />
-        <origin xyz="-0.39 -0.480 0.1" rpy="0 0 0" />
+        <origin xyz="-0.55 -0.480 0.1" rpy="0 0 0" />
         <axis xyz="0 1 0" />
     </joint>
@@ -109,5 +112,5 @@
         <parent link="base_link" />
         <child link="left_wheel_link" />
-        <origin xyz="-0.39 0.480 0.1" rpy="0 0 0" />
+        <origin xyz="-0.55 0.480 0.1" rpy="0 0 0" />
         <axis xyz="0 1 0" />
     </joint>
@@ -115,5 +118,5 @@
         <parent link="base_link" />
         <child link="back_right_wheel_link" />
-        <origin xyz="0.56 -0.480 0.1" rpy="0 0 0" />
+        <origin xyz="0.38 -0.480 0.1" rpy="0 0 0" />
         <axis xyz="0 1 0" />
     </joint>
@@ -121,5 +124,5 @@
         <parent link="base_link" />
         <child link="back_left_wheel_link" />
-        <origin xyz="0.56 0.480 0.1" rpy="0 0 0" />
+        <origin xyz="0.38 0.480 0.1" rpy="0 0 0" />
         <axis xyz="0 1 0" />
     </joint>
